File: KiCAD/TFT8K3548FPC-A1-E/TFT8K3548FPC-A1-E/TFT8K3548FPC-A1-E.kicad_pcb (KiCad board)
At the start: 2 copper layers, 49.4 x 89.2 mm, 24 parts, among them J1 TFT8K3548FPC-A1-E, J2 LCD_I8080_CONNECTOR_16x2, Q1 GP2302, U2 AMS1117-3.3

Commit message: lcd
Parts:
- added +1: LOGO, logo:monggoyun2, B.Cu at (124.7, 65.3)
