File: KiCAD/FH26W-45S-0.3SHW/FH26W-45S-0.3SHW/FH26W-45S-0.3SHW.sch (KiCad schematic (older format))
At the start: 28 parts, among them J1 NT35510-3.97inch-FH26W-45S-0.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, J2 LCD_I8080_CONNECTOR_16x2, U1 PT4103-SOT23-6, U2 AMS1117-3.3

Commit message: lcd
Parts:
- removed C5: C, Capacitor_SMD:C_0603_1608Metric_Pad1.05x0.95mm_HandSolder, symbol Device:C
- removed R3: 10K, Resistor_SMD:R_0603_1608Metric_Pad1.05x0.95mm_HandSolder, symbol Device:R
- removed TP6: +3.3V, TestPoint:TestPoint_Pad_2.5x2.5mm, symbol Connector:TestPoint
- removed TP7: GND, TestPoint:TestPoint_Pad_2.5x2.5mm, symbol Connector:TestPoint
- C3: value 0.1uF/25F -> 0.1uF/25V
- J2: symbol qconnectors:LCD_I8080_CONNECTOR_16x2 -> qconnectors:LCD_I8080_CONNECTOR_16x2-DIP
Connections:
- wire segments 129 -> 124
Changed lines of the file:
@@
 $EndDescr
 $Comp
-L qconnectors:LCD_I8080_CONNECTOR_16x2 J2
+L qconnectors:LCD_I8080_CONNECTOR_16x2-DIP J2
 U 1 1 5DD9A06E
 P 4550 3850
@@
 P 4600 1600
 F 0 "C3" V 4550 1450 50  0000 C CNN
-F 1 "0.1uF/25F" V 4550 1850 50  0000 C CNN
+F 1 "0.1uF/25V" V 4550 1850 50  0000 C CNN
 F 2 "Capacitor_SMD:C_0603_1608Metric_Pad1.05x0.95mm_HandSolder" H 4638 1450 50  0001 C CNN
 F 3 "~" H 4600 1600 50  0001 C CNN
@@
 Text Label 5100 1600 0    50   Italic 0
 GND
-$Comp
-L Device:R R3
-U 1 1 5DEEC1A3
-P 4250 3400
-F 0 "R3" V 4200 3200 50  0000 C CNN
-F 1 "10K" V 4250 3400 50  0000 C CNN
-F 2 "Resistor_SMD:R_0603_1608Metric_Pad1.05x0.95mm_HandSolder" V 4180 3400 50  0001 C CNN
-F 3 "~" H 4250 3400 50  0001 C CNN
-	1    4250 3400
-	0    1    1    0
-$EndComp
-Wire Wire Line
-	4400 3400 4850 3400
-$Comp
-L Device:C C5
-U 1 1 5DEFE26C
-P 5000 3400
-F 0 "C5" V 4950 3250 50  0000 C CNN
-F 1 "C" V 4950 3500 50  0000 C CNN
-F 2 "Capacitor_SMD:C_0603_1608Metric_Pad1.05x0.95mm_HandSolder" H 5038 3250 50  0001 C CNN
-F 3 "~" H 5000 3400 50  0001 C CNN
-	1    5000 3400
-	0    1    1    0
-$EndComp
-Wire Wire Line
-	5150 3400 5400 3400
-Text Label 3700 3400 0    50   Italic 0
-+3.3V
-Text Label 5200 3400 0    50   Italic 0
-GND
-Text Label 4550 3400 0    50   Italic 0
-RST
 $Comp
 L Device:R R4
@@
 Wire Wire Line
 	4400 3500 4850 3500
-Wire Wire Line
-	3650 3400 4100 3400
 Wire Wire Line
 	3650 3500 4100 3500
@@
 	0    -1   -1   0
 $EndComp
-$Comp
-L Connector:TestPoint TP6
-U 1 1 5DF6390E
-P 1850 4500
-F 0 "TP6" V 1900 4550 50  0000 C CNN
-F 1 "+3.3V" V 1850 4800 50  0000 C CNN
-F 2 "TestPoint:TestPoint_Pad_2.5x2.5mm" H 2050 4500 50  0001 C CNN
-F 3 "~" H 2050 4500 50  0001 C CNN
-	1    1850 4500
-	0    -1   -1   0
-$EndComp
-$Comp
-L Connector:TestPoint TP7
-U 1 1 5DF63B8F
-P 1850 4600
-F 0 "TP7" V 1900 4650 50  0000 C CNN
-F 1 "GND" V 1850 4900 50  0000 C CNN
-F 2 "TestPoint:TestPoint_Pad_2.5x2.5mm" H 2050 4600 50  0001 C CNN
-F 3 "~" H 2050 4600 50  0001 C CNN
-	1    1850 4600
-	0    -1   -1   0
-$EndComp
 Wire Wire Line
 	1850 4300 2150 4300
 Wire Wire Line
 	1850 4400 2150 4400
-Wire Wire Line
-	1850 4500 2150 4500
-Wire Wire Line
-	1850 4600 2150 4600
 Text Label 1900 4300 0    50   Italic 0
 LEDK
 Text Label 1900 4400 0    50   Italic 0
 +5V
-Text Label 1900 4500 0    50   Italic 0
-+3.3V
-Text Label 1900 4600 0    50   Italic 0
-GND
 $Comp
 L Connector:TestPoint TP11

Commit message: commit
Parts:
- added C5: 0.1uF, Capacitor_SMD:C_0603_1608Metric_Pad1.05x0.95mm_HandSolder, symbol Device:C
- added J3: I80 to RGB, Connector_FFC-FPC:Hirose_FH12-40S-0.5SH_1x40-1MP_P0.50mm_Horizontal, symbol Connector:Conn_01x40_Female
- added R6: 10K, Resistor_SMD:R_0603_1608Metric_Pad1.05x0.95mm_HandSolder, symbol Device:R
Connections:
- net labels added: +3V3, D10, D11, D12, D13, D14, D15, D18, D19, D2, D20, D21, D22, D23, D3, D4, D5, D6, D7, DE, HSYNC, LCD_CLK, VSYNC, X1, X2, Y1, Y2
- wire segments 124 -> 167
- no-connect marks 6 -> 9
