File: KiCAD/FH26W-45S-0.3SHW/FH26W-45S-0.3SHW/FH26W-45S-0.3SHW.kicad_pcb (KiCad board)
At the start: 2 copper layers, 70.5 x 97.8 mm, 28 parts, among them J1 NT35510-3.97inch-FH26W-45S-0.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, J2 LCD_I8080_CONNECTOR_16x2, U1 PT4103-SOT23-6, U2 AMS1117-3.3

Commit message: LCD
Other:
- board text added: "+5V"
- board text added: "BL"
- board text added: "D0"
- board text added: "D1"
- board text added: "D10"
- board text added: "D11"
- board text added: "D12"
- board text added: "D13"
- board text added: "D14"
- board text added: "D15"
- board text added: "D16"
- board text added: "D17"
- board text added: "D18"
- board text added: "D19"
- board text added: "D2"
- board text added: "D20"
- board text added: "D21"
- board text added: "D22"
- board text added: "D23"
- board text added: "D3"
- board text added: "D4"
- board text added: "D5"
- board text added: "D6"
- board text added: "D7"
- board text added: "D8"
- board text added: "D9"
- board text added: "GND"
- board text added: "RD"
- board text added: "RS"
- board text added: "RST"
- board text added: "WR"
- board text added: "~CS~"

Commit message: lcd
Parts:
- removed C5: C, Capacitor_SMD:C_0603_1608Metric_Pad1.05x0.95mm_HandSolder
- removed R3: 10K, Resistor_SMD:R_0603_1608Metric_Pad1.05x0.95mm_HandSolder
- removed TP6: +3.3V, TestPoint:TestPoint_Pad_2.5x2.5mm
- removed TP7: GND, TestPoint:TestPoint_Pad_2.5x2.5mm
- added G***: monggoyun2, logo:monggoyun2, B.Cu at (102.1, 80.7)
- C3: value 0.1uF/25F -> 0.1uF/25V
- moved J2 84.1 mm to (124.8, 33.1)
- moved R4 79.7 mm to (147.3, 41.0), turned to 0 degrees
- moved TP5 70.6 mm to (156.4, 72.4)
- moved D1 68.2 mm to (147.6, 85.9)
- moved L1 68.2 mm to (143.5, 91.7)
- moved U1 68.2 mm to (147.2, 91.8)
- moved R2 68.2 mm to (150.5, 92.4)
- moved R5 68.2 mm to (148.2, 88.3)
- moved R1 67.8 mm to (152.2, 92.4), turned to 90 degrees
- moved C2 65.5 mm to (151.1, 76.2), turned to 90 degrees
- moved TP4 63.3 mm to (156.4, 80.8)
- moved C1 63.3 mm to (140.8, 92.4), turned to 90 degrees
- moved TP3 62.7 mm to (156.4, 76.6)
- moved U2 55.6 mm to (145.8, 79.0), turned to 270 degrees
- moved C3 50.5 mm to (138.9, 92.3), turned to 270 degrees
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Connections:
- J2 pad 1: /~CS~ -> GND
- J2 pad 10: /DB4 -> /DB1
- J2 pad 11: /DB5 -> /DB2
- J2 pad 12: /DB6 -> /DB3
- J2 pad 13: /DB7 -> /DB4
- J2 pad 14: /DB8 -> /DB5
- J2 pad 15: /DB9 -> /DB6
- J2 pad 16: /DB10 -> /DB7
- J2 pad 17: /DB11 -> /DB8
- J2 pad 18: /DB12 -> /DB9
- J2 pad 19: /DB13 -> /DB10
- J2 pad 2: /RS -> +5V
- J2 pad 20: /DB14 -> /DB11
- J2 pad 21: /DB15 -> /DB12
- J2 pad 22: /DB16 -> /DB13
- J2 pad 23: /DB17 -> /DB14
- J2 pad 24: /DB18 -> /DB15
- J2 pad 25: /DB19 -> /DB16
- J2 pad 26: /DB20 -> /DB17
- J2 pad 27: /DB21 -> /DB18
- J2 pad 28: /DB22 -> /DB19
- J2 pad 29: /DB23 -> /DB20
- J2 pad 3: /WR -> /BL
- J2 pad 30: /BL -> /DB21
- J2 pad 31: +5V -> /DB22
- J2 pad 32: GND -> /DB23
- J2 pad 4: /RD -> /~CS~
- J2 pad 5: /RST -> /RS
- J2 pad 6: /DB0 -> /WR
- J2 pad 7: /DB1 -> /RD
- J2 pad 8: /DB2 -> /RST
- J2 pad 9: /DB3 -> /DB0
Routing:
- net GND: track 267.6 -> 18.7 mm, vias 10 -> 6
- net +3V3: track 209.2 -> 62.4 mm, vias 8 -> 3
- net /WR: track 92.2 -> 24.2 mm
- net /RST: track 83.6 -> 24.2 mm, vias 0 -> 2
- net /~CS~: track 85.1 -> 28.9 mm, vias 0 -> 3
- net /RD: track 72.1 -> 17.7 mm
- net /RS: track 70.8 -> 18.2 mm, vias 0 -> 2
- net /DB20: track 99.5 -> 47.3 mm
- net /DB22: track 102.4 -> 51.1 mm
- net /DB16: track 92.5 -> 43.5 mm
- net /DB18: track 95.0 -> 47.3 mm
- net /DB12: track 87.0 -> 39.7 mm
- net /DB8: track 82.3 -> 35.9 mm
- net /DB14: track 89.7 -> 43.5 mm
- net /DB6: track 81.6 -> 35.9 mm
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Other:
- outline, holes or cut-outs redrawn
- net class Default: clearance 0.2 -> 0.15; trace_width 0.25 -> 0.2
- rule trace_clearance: 0.2 -> 0.15
- rule trace_min: 0.2 -> 0.13

Commit message: OK 3.94 LCD
Routing:
- net GND: track 18.7 -> 27.3 mm, vias 6 -> 8
- net /WR: track 24.2 -> 22.0 mm
- net +3V3: track 62.4 -> 64.3 mm
- net /DB22: track 51.1 -> 52.9 mm
- net /DB8: track 35.9 -> 37.6 mm
- net /DB14: track 43.5 -> 45.1 mm
- net (no net): track 0.00 -> 1.56 mm
- net /DB18: track 47.3 -> 48.9 mm
- net /DB10: track 41.5 -> 42.9 mm
- net /DB6: track 35.9 -> 37.2 mm
- net /DB2: track 32.1 -> 33.2 mm
- net /RST: track 24.2 -> 25.1 mm
- net /TE: track 23.3 -> 22.5 mm
- net /DB12: track 39.7 -> 40.4 mm
- net /LEDK: track 70.0 -> 69.2 mm
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Other:
- net class Default: clearance 0.15 -> 0.13
- rule trace_clearance: 0.15 -> 0.13

Commit message: commit
Parts:
- added C5: 0.1uF, Capacitor_SMD:C_0603_1608Metric_Pad1.05x0.95mm_HandSolder, B.Cu at (149.0, 29.0)
- added J3: I80 to RGB, Connector_FFC-FPC:Hirose_FH12-40S-0.5SH_1x40-1MP_P0.50mm_Horizontal, B.Cu at (121.9, 75.4)
- added R6: 10K, Resistor_SMD:R_0603_1608Metric_Pad1.05x0.95mm_HandSolder, B.Cu at (149.0, 31.1)
Connections:
- net /DB0 renamed /D3
- net /DB1 renamed /D4
- net /DB10 renamed /D15
- net /DB11 renamed /D19
- net /DB12 renamed /D20
- net /DB13 renamed /D21
- net /DB14 renamed /D22
- net /DB15 renamed /D23
- net /DB2 renamed /D5
- net /DB3 renamed /D6
- net /DB4 renamed /D7
- net /DB5 renamed /D10
- net /DB6 renamed /D11
- net /DB7 renamed /D12
- net /DB8 renamed /D13
- net /DB9 renamed /D14
- net /RD renamed /HSYNC
- net /RS renamed /DE
- net /WR renamed /LCD_CLK
- net /~CS~ renamed /VSYNC
Routing:
- net /LEDK: track 69.2 -> 122.7 mm, vias 3 -> 5
- net +3V3: track 64.3 -> 112.2 mm, vias 3 -> 4
- net /DE: track 19.0 -> 62.2 mm, vias 2 -> 3
- net /LCD_CLK: track 22.0 -> 61.8 mm
- net /VSYNC: track 29.5 -> 67.8 mm, vias 3 -> 2
- net /D15: track 42.9 -> 78.2 mm
- net /LEDA: track 82.7 -> 117.6 mm
- net /HSYNC: track 18.1 -> 52.0 mm, vias 0 -> 3
- net /D5: track 33.2 -> 67.1 mm
- net /D11: track 37.2 -> 71.1 mm
- net /D20: track 40.4 -> 74.2 mm
- net /D22: track 45.1 -> 78.8 mm
- net /D13: track 37.6 -> 70.8 mm
- net /D3: track 28.8 -> 61.1 mm
- net /D7: track 32.7 -> 64.9 mm
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- added copper zone on B.Cu, net GND

Commit message: C100S
Parts:
- removed TP11, TP8: M3, MountingHole:MountingHole_3.2mm_M3_ISO14580_Pad
- removed TP3: LEDA, TestPoint:TestPoint_Pad_2.5x2.5mm
- removed TP4: LEDK, TestPoint:TestPoint_Pad_2.5x2.5mm
- added LEDA: LEDA, TestPoint:TestPoint_Pad_2.5x2.5mm, B.Cu at (147.9, 100.0)
- added LEDK: LEDK, TestPoint:TestPoint_Pad_2.5x2.5mm, B.Cu at (147.9, 104.2)
- moved ID 13.5 mm to (143.2, 66.0)
- moved TE 13.4 mm to (143.2, 62.2)
- moved 5V 9.77 mm to (146.7, 71.6)
- moved TP9 9.55 mm to (149.3, 126.0)
- moved TP10 9.42 mm to (99.0, 125.9)
- moved C2 0.85 mm to (150.3, 76.2)
- moved R1 0.72 mm to (151.5, 92.5)
- moved R2 0.58 mm to (149.9, 92.5)
- renumbered TP5 to 5V, TP2 to ID, TP1 to TE
Routing:
- net +5V: track 87.9 -> 83.3 mm, vias 4 -> 3
- net /LEDA: track 117.6 -> 121.6 mm
- net /BL: track 73.2 -> 69.8 mm
- net /LEDK: track 122.7 -> 126.0 mm, vias 5 -> 4
- net /TE: track 22.5 -> 24.0 mm
- net /LCD_ID: track 17.0 -> 15.6 mm, vias 2 -> 0
- net +3V3: track 112.2 -> 113.3 mm
Other:
- board size 70.5 x 97.8 mm -> 58 x 103.6 mm
- board text added: "JPJPJP"
