File: KiCAD/STM32F407VTE6-LCD/STM32F407VTE6-LCD/STM32F407VTE6-LCD.sch (KiCad schematic (older format))
At the start: 27 parts

Commit message: commit
Parts:
- added C? (x2): 22pF, symbol Device:C_Small
- added C? (x2): 0.1uF, symbol Device:C_Small
- added C? (x2): 10pF, symbol Device:C_Small
- added R? (x2): 1K, symbol Device:R
- added R? (x2): 22R, symbol Device:R
- added Y?: 32768Hz, symbol Device:Crystal_Small
- J?: footprint (none) -> qconnectors:NT35510-3.97inch-FH26W-45S-0.3SHW(60)_Handsoldering
- R?: value 10K -> 22R
- Y?: value Crystal_Small -> 8MHz
Connections:
- net labels added: DM, DP, OSC32_IN, OSC32_OUT, OSC_IN, OSC_OUT, SF_CLK, SF_MISO, SF_MOSI, SF_~CS~, SHIELD, TF_CLK, TF_CMD, TF_DAT0, TF_DAT1, TF_DAT2, TF_DAT3, USB_DET, USB_ID, VBUS
- net labels removed: PH0
- wire segments 182 -> 238
Other:
- moved on the sheet: D?, J?, U?, Y?
