File: KiCAD/RTD2831P-LQFP156/RTD2831P-LQFP156/RTD2831P-LQFP156.sch (KiCad schematic (older format))
At the start: 0 parts

Commit message: C100S
Changed lines of the file:
@@
 $EndDescr
 $Sheet
-S 2600 2800 1450 1100
+S 2900 2800 1450 1100
 U 5DEC7912
 F0 "POWER" 50
 F1 "POWER.sch" 50
+F2 "ST_5V" O R 4350 2850 50
+F3 "Vcore" O R 4350 2950 50
+F4 "STB_3V3" O R 4350 3050 50
+F5 "Vddr" O R 4350 3150 50
+F6 "+5V" O R 4350 3250 50
+F7 "+3V3" O R 4350 3350 50
+F8 "+1V8" O R 4350 3450 50
+F9 "GND" I R 4350 3550 50
+$EndSheet
+$Sheet
+S 7700 2800 1000 2650
+U 5DEC7CF7
+F0 "DISPLAY" 50
+F1 "DISPLAY.sch" 50
 $EndSheet
 $Sheet
@@
 F1 "CORE.sch" 50
 $EndSheet
-$Sheet
-S 7700 2800 1000 2650
-U 5DEC7CF7
-F0 "DISPLAY" 50
-F1 "DISPLAY.sch" 50
-$EndSheet
 $EndSCHEMATC
