File: KiCAD/STM32F407VTE6-SOCKET/STM32F407VTE6-SOCKET/STM32F407VTE6-SOCKET.kicad_pcb (KiCad board)
At the start: 2 copper layers, 45 x 84 mm, 42 parts, among them J1 USB_OTG, J2 Conn_02x20_Odd_Even, J3 Conn_02x20_Odd_Even, J4 Micro_SD_Card, J5 LCD_I8080_CONNECTOR_16x2-DIP, SW1 SW_MEC_5G, SW2 SW_MEC_5G, U1 TL431DBZ, U2 STM32F407VETx, U3 W25Q32JVZP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

Commit message: C100S
Parts:
- removed R9: 4K7, Resistor_SMD:R_0603_1608Metric_Pad1.05x0.95mm_HandSolder
- removed RST: SW_Push, Button_Switch_SMD:SW_SPST_FSMSM
- added C12: 2.2uF, Capacitor_SMD:C_0603_1608Metric_Pad1.05x0.95mm_HandSolder, B.Cu at (110.9, 143.6)
- added SW3: SW_Push, qmechanics:SW-Button-TS-018, F.Cu at (101.4, 169.5)
- U3: footprint Package_SON:WSON-8-1EP_6x5mm_P1.27mm_EP3.4x4.3mm -> qchip:GD5F1GQ4xBxIG_Handsoldering
- moved R10 3.88 mm to (120.9, 109.9)
- moved R12 3.88 mm to (122.5, 109.9)
- moved R11 3.87 mm to (124.1, 109.9)
- moved R13 3.86 mm to (125.6, 109.9)
- moved C8 2.78 mm to (125.0, 120.6)
- moved U3 1.61 mm to (123.8, 126.0)
- renumbered SWD to SWD1
Routing:
- net /NRST: track 15.6 -> 40.6 mm, vias 2 -> 3
- net +3V3: track 257.6 -> 248.0 mm, vias 18 -> 17
- net GNDREF: track 137.5 -> 130.1 mm, vias 36 -> 39
- net /B12: track 40.9 -> 46.0 mm
- net +5V: track 186.9 -> 191.2 mm
- net /A12: track 41.9 -> 37.8 mm
- net /A11: track 41.6 -> 37.5 mm
- net /A10: track 43.6 -> 39.7 mm
- net /A9: track 42.8 -> 38.9 mm
- net Net-(J1-Pad3): track 2.98 -> 6.83 mm
- net Net-(J1-Pad2): track 2.59 -> 6.44 mm
- net Net-(J1-Pad4): track 3.82 -> 7.20 mm
- net /B14: track 42.0 -> 44.4 mm
- net /DB4: track 41.6 -> 42.2 mm
- net /BL: track 74.7 -> 75.3 mm
