File: KiCAD/TFT8K3548FPC-A1-E-DIP/TFT8K3548FPC-A1-E-DIP/TFT8K3548FPC-A1-E-DIP.kicad_pcb (KiCad board)
At the start: 2 copper layers, 49.4 x 89.2 mm, 25 parts, among them J1 TFT8K3548FPC-A1-E, J2 LCD_I8080_CONNECTOR_16x2, Q1 GP2302, U2 AMS1117-3.3

Commit message: commit
Routing:
- net +3V3: track 105.7 -> 107.6 mm
- net GND: vias 7 -> 11
Changed lines of the file:
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@@
     (thickness 1.6)
     (drawings 45)
-    (tracks 278)
+    (tracks 283)
     (zones 0)
     (modules 25)
@@
   (page A4)
   (layers
-    (0 F.Cu signal hide)
+    (0 F.Cu signal)
     (31 B.Cu signal)
     (32 B.Adhes user)
@@
   (via (at 102.67 83.66) (size 0.8) (drill 0.4) (layers F.Cu B.Cu) (net 1))
   (segment (start 102.67 85.065) (end 102.67 83.66) (width 0.25) (layer B.Cu) (net 1))
+  (via (at 148.21 111.14) (size 1.21) (drill 1.2) (layers F.Cu B.Cu) (net 1))
+  (via (at 102.21 111.14) (size 1.21) (drill 1.2) (layers F.Cu B.Cu) (net 1))
+  (via (at 148.21 39.14) (size 1.21) (drill 1.2) (layers F.Cu B.Cu) (net 1))
+  (via (at 102.21 39.14) (size 1.21) (drill 1.2) (layers F.Cu B.Cu) (net 1))
   (segment (start 109.2 98.6) (end 111.2 98.6) (width 0.25) (layer F.Cu) (net 2))
   (segment (start 112.21 85.07) (end 112.21 81.18) (width 0.25) (layer B.Cu) (net 2))
@@
   (segment (start 129.27 85.07) (end 132.73 88.53) (width 0.25) (layer B.Cu) (net 2))
   (segment (start 114.1 85.07) (end 129.27 85.07) (width 0.25) (layer B.Cu) (net 2))
+  (segment (start 114.1 85.07) (end 112.21 85.07) (width 0.25) (layer B.Cu) (net 2))
   (segment (start 105.155 86.815) (end 105.16 86.81) (width 0.25) (layer B.Cu) (net 3))
   (segment (start 102.67 86.815) (end 105.155 86.815) (width 0.25) (layer B.Cu) (net 3))

Commit message: C100S
Parts:
- renumbered TP5 to +5V, TP6 to 3V3, TP7 to GND, TP2 to ID, TP3 to LEDA, TP4 to LEDK, TP1 to TE
Connections:
- J1 pad 17: /DB0 -> Net-(J1-Pad17)
- J1 pad 18: /DB1 -> /DB0
- J1 pad 19: /DB2 -> /DB1
- J1 pad 20: /DB3 -> /DB2
- J1 pad 21: /DB4 -> /DB3
- J1 pad 22: /DB5 -> /DB4
- J1 pad 23: /DB6 -> /DB5
- J1 pad 24: /DB7 -> /DB6
- J1 pad 25: /DB8 -> /DB7
- J1 pad 26: /DB9 -> Net-(J1-Pad26)
- J1 pad 27: /DB10 -> /DB8
- J1 pad 28: /DB11 -> /DB9
- J1 pad 29: /DB12 -> /DB10
- J1 pad 30: /DB13 -> /DB11
- J1 pad 31: /DB14 -> /DB12
- J1 pad 32: /DB15 -> /DB13
- J1 pad 33: /DB16 -> /DB14
- J1 pad 34: /DB17 -> /DB15
Routing:
- net /DB17: track 20.0 -> 0.00 mm
- net /DB16: track 16.9 -> 0.00 mm
- net /DB15: track 19.8 -> 19.1 mm
- net /DB8: track 16.0 -> 16.8 mm
- net /DB9: track 19.1 -> 19.7 mm
- net /DB14: track 16.7 -> 16.1 mm
Other:
- board text added: "0"
- board text added: "1"
- board text added: "16"
- board text added: "8"
- board text added: "JLCJLCJLC"
- board text added: "R1"
- board text added: "R2"
- board text added: "bit"
- board text removed: "D16"
- board text removed: "D17"
