File: KiCAD/TFT8K3548FPC-A1-E-DIP/TFT8K3548FPC-A1-E-DIP/TFT8K3548FPC-A1-E-DIP.sch (KiCad schematic (older format))
At the start: 25 parts, among them J1 TFT8K3548FPC-A1-E, J2 LCD_I8080_CONNECTOR_16x2, Q1 GP2302, U2 AMS1117-3.3

Commit message: commit
Changed lines of the file:
@@
 	1    0    0    -1
-$EndComp
-$Comp
-L Device:R R6
-U 1 1 5E058FF5
-P 7200 1650
-F 0 "R6" H 7150 1500 50  0000 C CNN
-F 1 "10K" V 7200 1650 50  0000 C CNN
-F 2 "Resistor_SMD:R_0603_1608Metric_Pad1.05x0.95mm_HandSolder" V 7130 1650 50  0001 C CNN
-F 3 "~" H 7200 1650 50  0001 C CNN
-	1    7200 1650
-	-1   0    0    1
 $EndComp
 Wire Wire Line
@@
 LEDA
 Wire Wire Line
-	7200 1850 7200 1800
-Wire Wire Line
 	7200 1400 7200 1450
 Connection ~ 7200 1450
 Wire Wire Line
 	7200 1450 7200 1500
-Wire Wire Line
-	7150 1850 7200 1850
-Wire Wire Line
-	7600 1850 7200 1850
 Text Label 7300 1850 0    50   Italic 0
 BL
@@
 	1    0    0    -1
 $EndComp
+Wire Wire Line
+	7600 1850 7200 1850
+Wire Wire Line
+	7150 1850 7200 1850
+$Comp
+L Device:R R6
+U 1 1 5E058FF5
+P 7200 1650
+F 0 "R6" H 7150 1500 50  0000 C CNN
+F 1 "10K" V 7200 1650 50  0000 C CNN
+F 2 "Resistor_SMD:R_0603_1608Metric_Pad1.05x0.95mm_HandSolder" V 7130 1650 50  0001 C CNN
+F 3 "~" H 7200 1650 50  0001 C CNN
+	1    7200 1650
+	-1   0    0    1
+$EndComp
+Wire Wire Line
+	7200 1850 7200 1800
+Connection ~ 7200 1850
 $EndSCHEMATC

Commit message: C100S
Connections:
- wire segments 122 -> 120
- no-connect marks 4 -> 6
Changed lines of the file:
@@
 	1450 1100 1800 1100
 Wire Wire Line
-	1450 2800 1800 2800
-Wire Wire Line
-	1450 3000 1800 3000
-Wire Wire Line
-	1450 3200 1800 3200
-Wire Wire Line
-	2600 3300 2950 3300
-Wire Wire Line
-	2600 3100 2950 3100
+	1450 2900 1800 2900
+Wire Wire Line
+	1450 3100 1800 3100
+Wire Wire Line
+	1450 3300 1800 3300
+Wire Wire Line
+	2600 3200 2950 3200
 Wire Wire Line
 	2600 2900 2950 2900
@@
 RST
 Text Label 2700 2300 0    50   Italic 0
-DB17
+DB15
 Text Label 2700 2500 0    50   Italic 0
-DB15
+DB13
 Text Label 2700 2700 0    50   Italic 0
-DB13
+DB11
+Text Label 1550 2800 0    50   Italic 0
+DB0
+Text Label 1550 3200 0    50   Italic 0
+DB4
+Text Label 2700 3000 0    50   Italic 0
+DB8
+Text Label 2700 2800 0    50   Italic 0
+DB10
 Text Label 2700 2900 0    50   Italic 0
-DB11
-Text Label 1550 2700 0    50   Italic 0
-DB0
+DB9
+Text Label 1550 2900 0    50   Italic 0
+DB1
 Text Label 1550 3100 0    50   Italic 0
-DB4
+DB3
 Text Label 1550 3300 0    50   Italic 0
-DB6
+DB5
 Text Label 2700 3200 0    50   Italic 0
-DB8
-Text Label 2700 3000 0    50   Italic 0
-DB10
-Text Label 2700 3100 0    50   Italic 0
-DB9
-Text Label 1550 2800 0    50   Italic 0
-DB1
-Text Label 1550 3000 0    50   Italic 0
-DB3
-Text Label 1550 3200 0    50   Italic 0
-DB5
-Text Label 2700 3300 0    50   Italic 0
 DB7
 Text Label 2700 1800 0    50   Italic 0
@@
 Text Label 1900 4950 0    50   Italic 0
 GND
-Text Label 1550 2900 0    50   Italic 0
+Text Label 1550 3000 0    50   Italic 0
 DB2
-Text Label 2700 2800 0    50   Italic 0
+Text Label 2700 2600 0    50   Italic 0
 DB12
-Text Label 2700 2600 0    50   Italic 0
+Text Label 2700 2400 0    50   Italic 0
 DB14
 Wire Wire Line
@@
 	1450 2300 1800 2300
 Wire Wire Line
+	2600 2400 2950 2400
+Wire Wire Line
 	2600 2600 2950 2600
 Wire Wire Line
@@
 	2600 3000 2950 3000
 Wire Wire Line
-	2600 3200 2950 3200
-Wire Wire Line
-	1450 3300 1800 3300
-Wire Wire Line
-	1450 3100 1800 3100
-Wire Wire Line
-	1450 2900 1800 2900
-Wire Wire Line
-	1450 2700 1800 2700
+	1450 3200 1800 3200
+Wire Wire Line
+	1450 3000 1800 3000
+Wire Wire Line
+	1450 2800 1800 2800
 Wire Wire Line
 	1450 1600 1800 1600
@@
 Text Label 2700 1100 0    50   Italic 0
 GND
-Wire Wire Line
-	2600 2400 2950 2400
-Text Label 2700 2400 0    50   Italic 0
-DB16
 Wire Wire Line
 	2600 1900 2950 1900
@@
 	7200 1850 7200 1800
 Connection ~ 7200 1850
+Wire Wire Line
+	2600 3300 2950 3300
+Text Label 2700 3300 0    50   Italic 0
+DB6
+NoConn ~ 1800 2700
+NoConn ~ 2600 3100
 $EndSCHEMATC
