File: KiCAD/TFT8K3548FPC-A1-E-DIP/TFT8K3548FPC-A1-E-DIP/TFT8K3548FPC-A1-E-DIP_1x2.kicad_pcb (KiCad board)
At the start: 2 copper layers, 99.4 x 89.2 mm, 50 parts, among them J1 TFT8K3548FPC-A1-E, J2 LCD_I8080_CONNECTOR_16x2, Q1 GP2302, U2 AMS1117-3.3

Commit message: C100S
Parts:
- removed TP1: TE, TestPoint:TestPoint_Pad_2.5x2.5mm
- removed TP2: LCD_ID, TestPoint:TestPoint_Pad_2.5x2.5mm
- removed TP3: LEDA, TestPoint:TestPoint_Pad_2.5x2.5mm
- removed TP4: LEDK, TestPoint:TestPoint_Pad_2.5x2.5mm
- removed TP5: +5V, TestPoint:TestPoint_Pad_2.5x2.5mm
- removed TP6: +3.3V, TestPoint:TestPoint_Pad_2.5x2.5mm
- removed TP7: GND, TestPoint:TestPoint_Pad_2.5x2.5mm
- added +5V: +5V, TestPoint:TestPoint_Pad_2.5x2.5mm, B.Cu at (54.3, 74.3)
- added 3V3: +3.3V, TestPoint:TestPoint_Pad_2.5x2.5mm, B.Cu at (54.3, 65.5)
- added GND: GND, TestPoint:TestPoint_Pad_2.5x2.5mm, B.Cu at (54.3, 70.0)
- added ID: LCD_ID, TestPoint:TestPoint_Pad_2.5x2.5mm, B.Cu at (60.6, 74.4)
- added LEDA: LEDA, TestPoint:TestPoint_Pad_2.5x2.5mm, B.Cu at (94.6, 83.7)
- added LEDK: LEDK, TestPoint:TestPoint_Pad_2.5x2.5mm, B.Cu at (94.5, 79.3)
- added TE: TE, TestPoint:TestPoint_Pad_2.5x2.5mm, B.Cu at (60.6, 70.1)
- renumbered TP5 to +5V, TP6 to 3V3, TP7 to GND, TP2 to ID, TP3 to LEDA, TP4 to LEDK, TP1 to TE
Connections:
- J1 pad 17: /DB0 -> Net-(J1-Pad17) (x2)
- J1 pad 18: /DB1 -> /DB0 (x2)
- J1 pad 19: /DB2 -> /DB1 (x2)
- J1 pad 20: /DB3 -> /DB2 (x2)
- J1 pad 21: /DB4 -> /DB3 (x2)
- J1 pad 22: /DB5 -> /DB4 (x2)
- J1 pad 23: /DB6 -> /DB5 (x2)
- J1 pad 24: /DB7 -> /DB6 (x2)
- J1 pad 25: /DB8 -> /DB7 (x2)
- J1 pad 26: /DB9 -> Net-(J1-Pad26) (x2)
- J1 pad 27: /DB10 -> /DB8 (x2)
- J1 pad 28: /DB11 -> /DB9 (x2)
- J1 pad 29: /DB12 -> /DB10 (x2)
- J1 pad 30: /DB13 -> /DB11 (x2)
- J1 pad 31: /DB14 -> /DB12 (x2)
- J1 pad 32: /DB15 -> /DB13 (x2)
- J1 pad 33: /DB16 -> /DB14 (x2)
- J1 pad 34: /DB17 -> /DB15 (x2)
Routing:
- net /DB17: track 40.1 -> 0.00 mm
- net /DB16: track 33.9 -> 0.00 mm
- net (no net): track 6.21 -> 0.00 mm
- net /DB15: track 39.7 -> 38.1 mm
- net /DB8: track 32.1 -> 33.6 mm
- net /DB9: track 38.3 -> 39.5 mm
- net /DB14: track 33.4 -> 32.3 mm
- net /DB3: track 39.2 -> 40.0 mm
- net /DB2: track 33.2 -> 34.1 mm
- net /DB7: track 38.3 -> 39.1 mm
- net /DB5: track 38.7 -> 39.5 mm
- net /DB4: track 32.8 -> 33.6 mm
- net /DB0: track 33.7 -> 34.5 mm
- net /DB1: track 39.6 -> 40.4 mm
- net /DB13: track 39.4 -> 38.6 mm
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Other:
- outline, holes or cut-outs redrawn
- board text added: "JPJPJP"
